File: hw/kicad/id=4_outdoor_pm/id=4_outdoor_pm.sch (KiCad schematic (older format))
At the start: 74 parts, among them IC1 LPS22HB, IC2 24AA02T-I_OT, IC3 SHTC1, IC4 LM3671MF-1.8_NOPB, IC5 SGP30-2.5k, IC6 24AA02T-I_OT, IC7 SN74AUP1T17DCKR, IC8 nRF52840-QIAA-T, J1 HDR_2x2.54mm, J2 53047-0810, Q1 NMOS_DGS, Q2 NMOS_DGS, Y1 32MHZ, Y2 32.768K

Commit message: Started with "Outdoor PM2.5 Module" schematic. Not finished yet.
Parts:
- removed C1, C12, C13, C16, C2, C22, C23, C26, C27, C28, C3, C30, C4, C6: 100nF, symbol C_Small
- removed C10, C11, C7, C8: 12pF, symbol C_Small
- removed C14, C5: 10uF, Capacitors_SMD:C_0805, symbol C_Small
- removed C15, C18: 1uF, symbol C_Small
- removed C17, C20: 1pF, symbol C_Small
- removed C19, C29: 4.7uF, symbol C_Small
- removed C21: 47nF, symbol C_Small
- removed C24, C32, C33: 100pF, symbol C_Small
- removed C25: 820pF, symbol C_Small
- removed C31: 10uF, symbol C_Small
- removed C9: 1.2pF, symbol C_Small
- removed D1: SD05T1G, SOD2512X110N, symbol SD05T1G
- removed D2: red, symbol LED_Small
- removed D3: green, symbol LED_Small
- removed IC1: LPS22HB, LGA10R50P2X3_200X200X80, symbol LPS22HB
- removed IC2, IC6: 24AA02T-I_OT, SOT95P270X145-5N, symbol 24AA02T-I_OT
- removed IC3: SHTC1, SON100P200X200X7500-5N, symbol SHTC1
- removed IC4: LM3671MF-1.8_NOPB, SOT95P280X145-5N, symbol LM3671MF-1.8_NOPB
- removed IC5: SGP30-2.5k, SON80P245X245X90-7N, symbol SGP30-2.5k
- removed IC7: SN74AUP1T17DCKR, SOT65P210X110-5N, symbol SN74AUP1T17DCKR
- removed IC8: nRF52840-QIAA-T, AQFN73, symbol nRF52840-QIAA-T
- removed J1: HDR_2x2.54mm, symbol Conn_01x02_Male
- removed J2: 53047-0810, SHDR8W35P0X125_1X8_1175X320X420P, symbol 53047-0810
- removed L1, L6, L7, L8, L9: 220Ohm@100MHz, symbol L
- removed L2: 2.2uH, symbol L
- removed L3: 3.9nH, symbol L
- removed L4: 15nH, symbol L
- removed L5: 10uH, symbol L
- removed Q1, Q2: NMOS_DGS, symbol Q_NMOS_DGS
- removed R1: 10M, symbol R
- removed R10, R11, R12, R13, R14, R15, R6, R7: 10k, symbol R_Small
- removed R2: 2M, symbol R
- removed R3, R4: 10k, symbol R
- removed R5: 12k, symbol R_Small
- removed R8, R9: 1k, symbol R_Small
- removed Y1: 32MHZ, FA128, symbol Q22FA12800025_FA-128_32_MHZ_8PF
- removed Y2: 32.768K, NX3215SA, symbol NX3215SA-32.768K-STD-MUA-9
- added C? (x10): 100nF, symbol C_Small
- added C?: 4.7uF, symbol C_Small
- added C? (x2): 1uF, symbol C_Small
- added C? (x4): 12pF, symbol C_Small
- added C? (x2): 1pF, symbol C_Small
- added C?: 1.2pF, symbol C_Small
- added C?: 820pF, symbol C_Small
- added C? (x3): 100pF, symbol C_Small
- added C?: 47nF, symbol C_Small
- added C?: 10uF, symbol C_Small
- added D?: green, symbol LED_Small
- added D?: red, symbol LED_Small
- added IC?: nRF52840-QIAA-T, AQFN73, symbol nRF52840-QIAA-T
- added IC?: LPS22HB, LGA10R50P2X3_200X200X80, symbol LPS22HB
- added IC?: 24AA02T-I_OT, SOT95P270X145-5N, symbol 24AA02T-I_OT
- added IC?: SN74AUP1T17DCKR, SOT65P210X110-5N, symbol SN74AUP1T17DCKR
- added IC?: SHT30-DIS-B, SON50P250X250X100-9N, symbol SHT30-DIS-B
- added J?: 53047-0810, SHDR8W35P0X125_1X8_1175X320X420P, symbol 53047-0810
- added L?: 10uH, symbol L
- added L?: 15nH, symbol L
- added L?: 3.9nH, symbol L
- added L? (x4): 220Ohm@100MHz, symbol L
- added Q? (x2): NMOS_DGS, symbol Q_NMOS_DGS
- added R? (x2): 10k, symbol R
- added R? (x2): 1k, symbol R_Small
- added R? (x8): 10k, symbol R_Small
- added R?: 12k, symbol R_Small
- added Y?: 32.768K, NX3215SA, symbol NX3215SA-32.768K-STD-MUA-9
- added Y?: 32MHZ, FA128, symbol Q22FA12800025_FA-128_32_MHZ_8PF
Connections:
- wire segments 229 -> 223
Other:
- note added: "Module ID = 4 --> Outdoor Partuculate Matter Module (PM2.5)"
- note removed: "Module ID = 3 --> Indoor Partuculate Matter Module (PM2.5, eCO2, VOC)"
- note removed: "Vdc_usb = 5V +/-0.5V (Imax = 0.5A)"
- note removed: "eCO2, VOC EEPROM"
- note removed: "eCO2, VOC Sensor"
